File: WeMos-TIC.brd (EAGLE design)
At the start: 33.2 x 25.7 mm, 22 parts, among them Q2 BSS138

Commit message: Bump to V1.1
Parts:
- removed D5: 1N4148, Seeed-Discrete:SOD123-2.7X1.6
- removed JP2: JUMPER-PAD-2-NC_BY_TRACE, SparkFun-Passives:PAD-JUMPER-2-NC_BY_TRACE_YES_SILK
- removed L1: WS2812B, _c2h:WS2812-PTH
- removed L2: WS2812B, _c2h:WS2812B-LONG
- removed U$1: PAD, _c2h:PAD-JUMPER-SWAP
- added D1: 1N4148, microbuilder:SOD-523
- added LED: WS2812-2020, SparkFun-LED:WS2812-2020
- added R6: 1K, _c2h:0603-RES
- added RX: TIC-RX, SparkFun-Jumpers:SMT-JUMPER_3_1-NC_TRACE_SILK
- added TIC: (no value), _c2h:0603-LED
- C1: device _c2h:0805-CAP -> _c2h:0402-CAP-OK
- R1, R2, R5: device _c2h:0805-RES -> _c2h:0603-RES
- R3: value 1.2K -> 220; device _c2h:0805-RES -> _c2h:0603-RES
- R4: value 10k -> 3K3; device _c2h:0805-RES -> _c2h:0603-RES
- moved R3 16.8 mm to (15.7, 15.7)
- moved C1 15.4 mm to (30.8, 4.76), turned to 180 degrees
- moved R5 9.97 mm to (17.5, 8.45)
- moved Q2 6.52 mm to (15.7, 12.7), turned to 270 degrees
- moved OK1 6.35 mm to (10.2, 12.7)
- moved R4 5.91 mm to (14.7, 8.45), turned to 90 degrees
- moved R1 3.26 mm to (3.30, 19.1), turned to 180 degrees
- moved TINFO 3.18 mm to (26.0, 12.7)
- moved R2 1.29 mm to (5.65, 12.8)
Connections:
- net MISO renamed GPIO12
- removed net MOSI: JP3.6, JP7.6
- removed net N$6: L1.4, L2.2
- removed net SCK: JP3.4, JP7.4, L1.1, L2.4
- removed net V+O: I2C_OLED1.1, U$1.3
- removed net V-O: I2C_OLED1.2, U$1.2
- new net GPIO13: JP3.6, JP7.6, RX.3
- new net GPIO14: JP3.4, JP7.4, LED.3
- new net N$1: R6.2, TIC.MINUS
- new net TIC-RX: Q2.3, R5.1, R6.1, RX.2
- net 3V3: now also I2C_OLED1.2, JP5.2, TIC.PLUS; no longer U$1.4, U$1.44
- net 5V: now also D1.A, JP5.1; no longer D5.1, JP2.2
- net GND: now also I2C_OLED1.1, LED.2; no longer JP5.1, JP5.2, L1.3, L2.3, U$1.1, U$1.11
- net GPIO3: now also RX.1; no longer Q2.3, R5.1
- net VLED: now also D1.K, LED.4; no longer D5.2, JP2.1, L1.2, L2.1
Routing:
- net 3V3: track 49.6 -> 76.7 mm, vias 0 -> 1
- net 5V: track 28.1 -> 47.1 mm
- net GPIO3: track 30.6 -> 12.2 mm
- net TIC-RX: track 0.00 -> 15.7 mm
- net GPIO14: track 0.00 -> 15.7 mm
- net GPIO13: track 0.00 -> 15.0 mm
- net SCK: track 14.4 -> 0.00 mm
- net N$3: track 20.6 -> 7.99 mm
- net N$5: track 5.43 -> 15.8 mm, vias 0 -> 1
- net V-O: track 9.00 -> 0.00 mm
- net V+O: track 6.95 -> 0.00 mm
- net N$4: track 12.7 -> 17.6 mm
- net N$2: track 9.39 -> 13.0 mm
- net VLED: track 9.85 -> 6.53 mm
- net N$1: track 0.00 -> 3.24 mm
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Other:
- board text added: "IO13"
- board text added: "IO3"
- board text added: "V1.1"
- board text added: "hallard.me/teleinfo"
- board text removed: "V1.0"

Commit message: Bump to v1.2
Parts:
- removed JP7, JP8: (no value), SparkFun-Connectors:1X08_NO_SILK
- removed Q2: BSS138, Seeed-Discrete:SOT23
- removed TINFO: 1X2-3.5MM, adafruit:1X2-3.5MM
- removed U$2: (no value), _c2h:LOGO_C2I_015
- added J1: KF2EDGR-3.81-2P, _c2h:1X2-3.5MM
- added J2: Qwiic Connector, _c2h:JST04_1MM_VERT
- added JLED: (no value), SparkFun-Passives:PAD-JUMPER-2-NC_BY_TRACE_YES_SILK
- added Q1: BSS138, _c2h:SOT-323-3
- R1, R2, R4, R5, R6: device _c2h:0603-RES -> _c2h:0402-RES
- R3: value 220 -> 2K; device _c2h:0603-RES -> adafruit:TC33X
- TIC: value (none) -> BLUE; device _c2h:0603-LED -> OPL_Optoelectronics:LED-0402
- moved R2 4.93 mm to (6.67, 7.94), turned to 0 degrees
- moved R4 2.61 mm to (16.7, 10.2), turned to 180 degrees
- moved R1 2.53 mm to (5.71, 18.3), turned to 90 degrees
- moved R3 2.17 mm to (17.8, 16.5), turned to 90 degrees
- moved RX 1.91 mm to (21.6, 12.7)
- moved OK1 1.90 mm to (12.1, 12.7)
- moved R5 1.00 mm to (16.7, 7.87), turned to 180 degrees
- moved TIC 0.06 mm to (30.5, 19.1), turned to 180 degrees
Connections:
- new net LTIC: JLED.2, TIC.+
- net 3V3: now also J2.2, JLED.1; no longer JP7.8, TIC.PLUS
- net 5V: no longer JP8.8
- net A0: no longer JP7.2
- net GND: now also J2.1, Q1.2; no longer JP8.7, Q2.2
- net GPIO0: no longer JP8.5
- net GPIO1: no longer JP8.1
- net GPIO12: no longer JP7.5
- net GPIO13: no longer JP7.6
- net GPIO14: no longer JP7.4
- net GPIO16: no longer JP7.3
- net GPIO2: no longer JP8.6
- net GPIO3: no longer JP8.2
- net N$1: now also TIC.-; no longer TIC.MINUS
- net N$2: now also Q1.1; no longer Q2.1
- net N$4: now also J1.1; no longer TINFO.1
- net N$5: now also J1.2; no longer TINFO.2
- net RST: no longer JP7.1
- net SCL: now also J2.4; no longer JP8.3
- net SDA: now also J2.3; no longer JP8.4
- net SS: no longer JP7.7
- net TIC-RX: now also Q1.3; no longer Q2.3
Routing:
- net SCL: track 27.1 -> 34.1 mm, vias 0 -> 1
- net LTIC: track 0.00 -> 6.56 mm, vias 0 -> 1
- net SDA: track 23.0 -> 27.9 mm, vias 0 -> 1
- net N$3: track 7.99 -> 11.8 mm
- net SS: track 2.54 -> 0.00 mm
- net RST: track 2.54 -> 0.00 mm
- net GPIO16: track 2.54 -> 0.00 mm
- net GPIO12: track 2.54 -> 0.00 mm
- net A0: track 2.54 -> 0.00 mm
- net GPIO2: track 2.54 -> 0.00 mm
- net GPIO1: track 2.54 -> 0.00 mm
- net GPIO0: track 2.54 -> 0.00 mm
- net GND: track 2.54 -> 0.00 mm, vias 12 -> 16
- net N$5: track 15.8 -> 13.8 mm
- net N$4: track 17.6 -> 15.7 mm
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Other:
- board text added: "1"
- board text added: "10"
- board text added: "11"
- board text added: "17"
- board text added: "18"
- board text added: "19"
- board text added: "21"
- board text added: "22"
- board text added: "23"
- board text added: "26"
- board text added: "3"
- board text added: "32-C3"
- board text added: "32-S2"
- board text added: "32-S3"
- board text added: "33"
- board text added: "35"
- board text added: "36"
- board text added: "6"
- board text added: "7"
- board text added: "8"
- board text added: "8266"
- board text added: "9"
- board text added: "Cut to disable Teleinfo LED"
- board text added: "EN"
- board text added: "ESP"
- board text added: "ESP32"
- board text added: "J2"
- board text added: "SVP"
- board text added: "V1.2"
- board text added: "hallard.me"
- board text removed: "IO13"
- board text removed: "IO3"
- board text removed: "V1.1"
